Commit message: [fetch_description] temporary change to convert model to VRML with simtrans.

File: fetch_description/robots/fetch.urdf (robot description, URDF)
Before this commit: robot fetch, 26 links, 25 joints
Links:
- link estop_link: geometry collision mesh filename=package://fetch_description/meshes/estop_link.STL; visual mesh filename=package://fetch_description/meshes/estop_link.STL
